Commit message: urdf update

File: src/vehicle_launch/config/robot.urdf.xacro (robot description, xacro)
@@ -9,5 +9,5 @@
     <origin xyz="0 0 0" rpy="0 0 0" />
   </joint>
-  <link name="velodyne"> </link>
+  <link name="os_sensor"> </link>
   <joint name="lidar_joint" type="fixed">
     <parent link="chassis_link" />

Commit message: urdf update

File: src/vehicle_launch/config/robot.urdf.xacro (robot description, xacro)
@@ -12,5 +12,5 @@
   <joint name="lidar_joint" type="fixed">
     <parent link="chassis_link" />
-    <child link="velodyne" />
+    <child link="os_sensor" />
     <origin xyz="0 0 1.1" rpy="0 0 0" />
   </joint>
